File: resources/pcba/booster/booster.kicad_pcb (KiCad board)
At the start: 2 copper layers, 44 x 64 mm, 41 parts, among them J1 LED, J2 PSU, J3 ESP, Q1 IRLML0030, Q2 PMOS 9301, Q3 VOM1271T, Q4 IRLML0030, U1 ADuM1200BR, U2 CD4051B, U3 L78L05_SOT89, U4 MCP6001-OT, U5 ADuM1200BR

Commit message: update booster kicad lib
Parts:
- Q3: footprint VOM1271T:SOP-4_VIS -> trypillia:VOM1271T
Changed lines of the file:
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@@
 		(0 "F.Cu" signal)
 		(2 "B.Cu" signal)
-		(5 "F.SilkS" user)
-		(7 "B.SilkS" user)
+		(5 "F.SilkS" user "F.Silkscreen")
+		(7 "B.SilkS" user "B.Silkscreen")
 		(1 "F.Mask" user)
 		(3 "B.Mask" user)
 		(25 "Edge.Cuts" user)
 		(27 "Margin" user)
-		(31 "F.CrtYd" user)
-		(29 "B.CrtYd" user)
+		(31 "F.CrtYd" user "F.Courtyard")
+		(29 "B.CrtYd" user "B.Courtyard")
 	)
 	(setup
@@
 		)
 		(property ki_fp_filters "R_*")
-		(sheetname "PSU")
+		(sheetname "/PSU/")
 		(sheetfile "psu.kicad_sch")
 		(attr smd)
@@
 		)
 		(property ki_fp_filters "R_*")
-		(sheetname "PSU")
+		(sheetname "/PSU/")
 		(sheetfile "psu.kicad_sch")
 		(attr smd)
@@
 		)
 		(property ki_fp_filters "SOT?23*")
-		(sheetname "PSU")
+		(sheetname "/PSU/")
 		(sheetfile "psu.kicad_sch")
 		(attr smd)
@@
 		)
 		(property ki_fp_filters "D*DO?41*")
-		(sheetname "PSU")
+		(sheetname "/PSU/")
 		(sheetfile "psu.kicad_sch")
 		(attr smd)
@@
 		)
 		(property ki_fp_filters "R_*")
-		(sheetname "PSU")
+		(sheetname "/PSU/")
 		(sheetfile "psu.kicad_sch")
 		(attr smd)
@@
 		)
 		(property ki_fp_filters "SOT?23*")
-		(sheetname "PSU")
+		(sheetname "/PSU/")
 		(sheetfile "psu.kicad_sch")
 		(attr smd)
@@
 		)
 		(property ki_fp_filters "R_*")
-		(sheetname "PSU")
+		(sheetname "/PSU/")
 		(sheetfile "psu.kicad_sch")
 		(attr smd)
@@
 		)
 		(property ki_fp_filters "R_*")
-		(sheetname "PSU")
+		(sheetname "/PSU/")
 		(sheetfile "psu.kicad_sch")
 		(attr smd)
@@
 		)
 		(property ki_fp_filters "R_*")
-		(sheetname "PSU")
+		(sheetname "/PSU/")
 		(sheetfile "psu.kicad_sch")
 		(attr smd)
@@
 		)
 		(property ki_fp_filters "R_*")
-		(sheetname "PSU")
+		(sheetname "/PSU/")
 		(sheetfile "psu.kicad_sch")
 		(attr smd)
@@
 		)
 		(property ki_fp_filters "R_*")
-		(sheetname "PSU")
+		(sheetname "/PSU/")
 		(sheetfile "psu.kicad_sch")
 		(attr smd)
@@
 		)
 		(property ki_fp_filters "Connector*:*_1x??_*")
-		(sheetname "PSU")
+		(sheetname "/PSU/")
 		(sheetfile "psu.kicad_sch")
 		(attr through_hole)
@@
 		)
 		(property ki_fp_filters "SOT?89*")
-		(sheetname "PSU")
+		(sheetname "/PSU/")
 		(sheetfile "psu.kicad_sch")
 		(attr smd)
@@
 		)
 		(property ki_fp_filters "R_*")
-		(sheetname "PSU")
+		(sheetname "/PSU/")
 		(sheetfile "psu.kicad_sch")
 		(attr smd)
@@
 		)
 		(property ki_fp_filters "R_*")
-		(sheetname "PSU")
+		(sheetname "/PSU/")
 		(sheetfile "psu.kicad_sch")
 		(attr smd)
@@
 		)
 		(property ki_fp_filters "R_*")
-		(sheetname "PSU")
+		(sheetname "/PSU/")
 		(sheetfile "psu.kicad_sch")
 		(attr smd)
@@
 		)
 	)
-	(footprint "VOM1271T:SOP-4_VIS"
+	(footprint "trypillia:VOM1271T"
 		(layer "F.Cu")
 		(at 95.13 101.55 90)
@@
 		)
 		(property ki_fp_filters "SOP-4_VIS SOP-4_VIS-M SOP-4_VIS-L")
-		(sheetname "PSU")
+		(sheetname "/PSU/")
 		(sheetfile "psu.kicad_sch")
 		(attr smd)
@@
 		)
 		(embedded_fonts no)
-		(model "/Users/stasstarcha/Documents/dobrotvir/3dmodels/VOM1271T/SOP-4V2.step"
+		(model "${KIPRJMOD}/lib/3dmodels/VOM1271-SOP-4.step"
 			(offset
 				(xyz 0 0 1.1)
@@
 		)
 		(property ki_fp_filters "R_*")
-		(sheetname "PSU")
+		(sheetname "/PSU/")
 		(sheetfile "psu.kicad_sch")
 		(attr smd)
@@
 		)
 		(property ki_fp_filters "R_*")
-		(sheetname "PSU")
+		(sheetname "/PSU/")
 		(sheetfile "psu.kicad_sch")
 		(attr smd)
@@
 		)
 		(property ki_fp_filters "R_*")
-		(sheetname "PSU")
+		(sheetname "/PSU/")
 		(sheetfile "psu.kicad_sch")
 		(attr smd)
@@
 		)
 		(property ki_fp_filters "R_*")
-		(sheetname "PSU")
+		(sheetname "/PSU/")
 		(sheetfile "psu.kicad_sch")
 		(attr smd)
@@
 		)
 		(property ki_fp_filters "C_*")
-		(sheetname "PSU")
+		(sheetname "/PSU/")
 		(sheetfile "psu.kicad_sch")
 		(attr smd)
@@
 		)
 		(property ki_fp_filters "R_*")
-		(sheetname "PSU")
+		(sheetname "/PSU/")
 		(sheetfile "psu.kicad_sch")
 		(attr smd)
@@
 		)
 		(property ki_fp_filters "R_*")
-		(sheetname "PSU")
+		(sheetname "/PSU/")
 		(sheetfile "psu.kicad_sch")
 		(attr smd)
@@
 		)
 		(property ki_fp_filters "R_*")
-		(sheetname "PSU")
+		(sheetname "/PSU/")
 		(sheetfile "psu.kicad_sch")
 		(attr smd)
@@
 		)
 		(property ki_fp_filters "TSSOP*4.4x5mm*P0.65mm* DIP*W7.62* SOIC*3.9x9.9mm*P1.27mm* SO*5.3x10.2mm*P1.27mm*")
-		(sheetname "PSU")
+		(sheetname "/PSU/")
 		(sheetfile "psu.kicad_sch")
 		(attr smd)
@@
 		)
 		(property ki_fp_filters "SOT?23*")
-		(sheetname "PSU")
+		(sheetname "/PSU/")
 		(sheetfile "psu.kicad_sch")
 		(attr smd)
@@
 		)
 		(property ki_fp_filters "Connector*:*_1x??_*")
-		(sheetname "PSU")
+		(sheetname "/PSU/")
 		(sheetfile "psu.kicad_sch")
 		(attr through_hole)
@@
 		)
 		(property ki_fp_filters "C_*")
-		(sheetname "PSU")
+		(sheetname "/PSU/")
 		(sheetfile "psu.kicad_sch")
 		(attr smd)
@@
 		)
 		(property ki_fp_filters "SOIC*3.9x4.9mm*P1.27mm*")
-		(sheetname "PSU")
+		(sheetname "/PSU/")
 		(sheetfile "psu.kicad_sch")
 		(attr smd)
@@
 		)
 		(property ki_fp_filters "C_*")
-		(sheetname "PSU")
+		(sheetname "/PSU/")
 		(sheetfile "psu.kicad_sch")
 		(attr smd)
@@
 		)
 		(property ki_fp_filters "R_*")
-		(sheetname "PSU")
+		(sheetname "/PSU/")
 		(sheetfile "psu.kicad_sch")
 		(attr smd)
@@
 		)
 		(property ki_fp_filters "R_*")
-		(sheetname "PSU")
+		(sheetname "/PSU/")
 		(sheetfile "psu.kicad_sch")
 		(attr smd)
@@
 		)
 		(property ki_fp_filters "SOIC*3.9x4.9mm*P1.27mm*")
-		(sheetname "PSU")
+		(sheetname "/PSU/")
 		(sheetfile "psu.kicad_sch")
 		(attr smd)
@@
 		)
 		(property ki_fp_filters "Connector*:*_1x??_*")
-		(sheetname "PSU")
+		(sheetname "/PSU/")
 		(sheetfile "psu.kicad_sch")
 		(attr through_hole)
@@
 		)
 		(property ki_fp_filters "R_*")
-		(sheetname "PSU")
+		(sheetname "/PSU/")
 		(sheetfile "psu.kicad_sch")
 		(attr smd)
@@
 		)
 		(property ki_fp_filters "R_*")
-		(sheetname "PSU")
+		(sheetname "/PSU/")
 		(sheetfile "psu.kicad_sch")
 		(attr smd)
@@
 		)
 		(property ki_fp_filters "C_*")
-		(sheetname "PSU")
+		(sheetname "/PSU/")
 		(sheetfile "psu.kicad_sch")
 		(attr smd)
@@
 		)
 		(property ki_fp_filters "SOT?23*")
-		(sheetname "PSU")
+		(sheetname "/PSU/")
 		(sheetfile "psu.kicad_sch")
 		(clearance 0.1)
@@
 		)
 		(property ki_fp_filters "R_*")
-		(sheetname "PSU")
+		(sheetname "/PSU/")
 		(sheetfile "psu.kicad_sch")
 		(attr smd)
@@
 		)
 		(property ki_fp_filters "C_*")
-		(sheetname "PSU")
+		(sheetname "/PSU/")
 		(sheetfile "psu.kicad_sch")
 		(attr smd)
