File: resources/pcba/booster/psu.kicad_sch (KiCad schematic)
At the start: 41 parts, among them J1 LED, J2 PSU, J3 ESP, Q1 IRLML0030, Q2 PMOS 9301, Q3 VOM1271T, Q4 IRLML0030, U1 ADuM1200BR, U2 CD4051B, U3 L78L05_SOT89, U4 MCP6001-OT, U5 ADuM1200BR

Commit message: update booster kicad lib
Parts:
- Q3: footprint SOP-4_VIS -> trypillia:VOM1271T
Changed lines of the file:
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@@
 			)
 		)
-		(property "Footprint" "SOP-4_VIS"
+		(property "Footprint" "trypillia:VOM1271T"
 			(at 45.72 172.72 0)
 			(effects
