File: resources/pcba/core/core.kicad_pcb (KiCad board)
At the start: 2 copper layers, 94 x 70 mm, 77 parts, among them J1 PSU BTN, J10 INV LOAD, J11 RS485, J12 FAN, J13 BMS UART, J14 UART0, J2 USB, J3 ATS, J4 DISPLAY, J5 Buzzer, J6 PSU A, J7 PSU B, J8 BAT, J9 INV BTN, Q1 PMOS IPD042P03L3, SW1 RST, SW2 BOOT, U1 AMS1117-3.3, U10 L7805, U11 L7805, U12 ADuM1201BR, U13 USBLC6-2SC6, U2 ESP32-S3-WROOM-1, U3 B0505S, U4 LM2596S-ADJ, U5 EL357N, U6 ADuM1201BR, U7 74LVC1G04, U8 MAX485E, U9 ADuM1200BR

Commit message: update ble protocol
Parts:
- R17, R18: value 4.7k -> 10k
Changed lines of the file:
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@@
 			)
 		)
-		(property "Value" "4.7k"
+		(property "Value" "10k"
 			(at 0 1.82 0)
 			(layer "F.Fab")
@@
 			)
 		)
-		(property "Value" "4.7k"
+		(property "Value" "10k"
 			(at 0 1.82 0)
 			(layer "F.Fab")
